File: electronics/main.kicad_sch (KiCad schematic)
At the start: 12 parts, among them J5 Conn_01x02_Socket, J6 Conn_01x02_Socket, J7 Conn_01x02_Socket, J8 Conn_01x02_Socket, SW1 SW_SPDT, U1 XIAO-ESP32-C6-SMD, U2 TLC5917QDRQ1

Commit message: [WIP] in prgress, copy real circuit..
Parts:
- removed D1: LED, LED_THT:LED_D5.0mm, symbol Device:LED
- removed J-batt1, J5, J6, J7, J8: Conn_01x02_Socket, Library:Molex_PicoBlade_53048-0210_1x02_P1.25mm_Horizontal_2, symbol Connector:Conn_01x02_Socket
- added D2: LED_RKBG, LED_THT:LED_D5.0mm-4_RGB, symbol Device:LED_RKBG
- added J1, J2, J3, J4, J9: Conn_01x03_Socket, Connector_Molex:Molex_PicoBlade_53048-0310_1x03_P1.25mm_Horizontal, symbol Connector:Conn_01x03_Socket
- added R3: 150, Resistor_THT:R_Axial_DIN0207_L6.3mm_D2.5mm_P10.16mm_Horizontal, symbol Device:R
- R2: value 470 -> 22
Connections:
- net +BATT: now also J1.1 (Pin_1), J2.1 (Pin_1), J3.1 (Pin_1), J4.1 (Pin_1); no longer R2.1
- net GND: now also D2.2 (K), J9.1 (Pin_1)
- net at R2.2: now also D2.4 (GA)
- net at SW1.2 (B), SW1.3 (C): now also J9.3 (Pin_3)
- net at U1.1 (GPIO0_A0_D0): now also R3.1
- net at U1.2 (GPIO1_A1_D1): now also R2.1
- net at U2.11 (OUT6): now also J3.3 (Pin_3)
- net at U2.10 (OUT5): now also J2.3 (Pin_3)
- net at U2.12 (OUT7): now also J4.3 (Pin_3)
- net at U2.9 (OUT4): now also J1.3 (Pin_3)
- new net: D2.1 (RA), R3.2
Other:
- moved on the sheet: R2

Commit message: [WIP] 青色LEDで動作確認まで完了
Parts:
- added R4, R5: 22, Resistor_THT:R_Axial_DIN0207_L6.3mm_D2.5mm_P10.16mm_Horizontal, symbol Device:R
Connections:
- net +BATT: now also R4.1
- net GND: now also R5.2
- net at J1.3 (Pin_3): now also U2.11 (OUT6); no longer U2.9 (OUT4)
- net at R2.1: now also U1.6 (GPIO23_D5_SCL); no longer U1.2 (GPIO1_A1_D1)
- net at J2.3 (Pin_3): now also U2.12 (OUT7); no longer U2.10 (OUT5)
- net at U1.1 (GPIO0_A0_D0): now also R4.2, R5.1; no longer R3.1
- net at U1.5 (GPIO22_D4_SDA): now also R3.1
- net at J4.3 (Pin_3): now also U2.9 (OUT4); no longer U2.12 (OUT7)
- net at J3.3 (Pin_3): now also U2.10 (OUT5); no longer U2.11 (OUT6)
Other:
- moved on the sheet: J1, J2, J3, J4

Commit message: [ele] v2 layout draft
Parts:
- removed J1, J2, J3, J4: Conn_01x03_Socket, Connector_Molex:Molex_PicoBlade_53048-0310_1x03_P1.25mm_Horizontal, symbol Connector:Conn_01x03_Socket
- added J1, J2, J3, J4, J5, J6, J7, J8: Conn_01x02_Socket, Connector_Molex:Molex_PicoBlade_53048-0210_1x02_P1.25mm_Horizontal, symbol Connector:Conn_01x02_Socket
- R1, R4, R5: footprint Resistor_THT:R_Axial_DIN0207_L6.3mm_D2.5mm_P10.16mm_Horizontal -> Resistor_SMD:R_0603_1608Metric_Pad0.98x0.95mm_HandSolder
- RV1: footprint Snapeda:TRIM_3362P-1-103 -> Potentiometer_SMD:Potentiometer_Bourns_TC33X_Vertical
Connections:
- net +BATT: now also J1.1 (Pin_1), J2.1 (Pin_1), J3.1 (Pin_1), J4.1 (Pin_1), J5.1 (Pin_1), J6.1 (Pin_1), J7.1 (Pin_1), J8.1 (Pin_1)
- net at U2.11 (OUT6): now also J7.2 (Pin_2)
- net at R1.1, RV1.1: now also RV1.2
- net at RV1.3, U2.15 (R-EXT): no longer RV1.2
- net at U2.12 (OUT7): now also J8.2 (Pin_2)
- net at U2.9 (OUT4): now also J5.2 (Pin_2)
- net at U2.10 (OUT5): now also J6.2 (Pin_2)
- net at U2.5 (OUT0): now also J1.2 (Pin_2)
- net at U2.6 (OUT1): now also J2.2 (Pin_2)
- net at U2.7 (OUT2): now also J3.2 (Pin_2)
- net at U2.8 (OUT3): now also J4.2 (Pin_2)

Commit message: [WIP]
Connections:
- net GND: now also U2.14 (SDO)
- net at U1.10 (GPIO20_D9_MISO): no longer U2.14 (SDO)
Changed lines of the file:
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@@
-	(wire
-		(pts
-			(xy 91.44 81.28) (xy 119.38 81.28)
-		)
-		(stroke
-			(width 0)
-			(type default)
-		)
-	)
 	(wire
 		(pts
@@
 	(wire
 		(pts
+			(xy 121.92 82.55) (xy 121.92 80.01)
+		)
+		(stroke
+			(width 0)
+			(type default)
+		)
+	)
+	(wire
+		(pts
 			(xy 40.64 82.55) (xy 40.64 85.09)
 		)
@@
 	(wire
 		(pts
-			(xy 119.38 81.28) (xy 119.38 80.01)
-		)
-		(stroke
-			(width 0)
-			(type default)
-		)
-	)
-	(wire
-		(pts
 			(xy 17.78 95.25) (xy 20.32 95.25)
-		)
-		(stroke
-			(width 0)
-			(type default)
-		)
-	)
-	(wire
-		(pts
-			(xy 119.38 80.01) (xy 121.92 80.01)
 		)
 		(stroke
@@
 					(unit 1)
 				)
+			)
+		)
+	)
+	(symbol
+		(lib_id "power:GND")
+		(at 121.92 82.55 0)
+		(unit 1)
+		(exclude_from_sim no)
+		(in_bom yes)
+		(on_board yes)
+		(dnp no)
+		(property "Reference" "#PWR011"
+			(at 121.92 88.9 0)
+			(effects
+				(font
+					(size 1.27 1.27)
+				)
+				(hide yes)
+			)
+		)
+		(property "Value" "GND"
+			(at 123.19 87.63 0)
+			(effects
+				(font
+					(size 1.27 1.27)
+				)
+			)
+		)
+		(property "Footprint" ""
+			(at 121.92 82.55 0)
+			(effects
+				(font
+					(size 1.27 1.27)
+				)
+				(hide yes)
+			)
+		)
+		(property "Datasheet" ""
+			(at 121.92 82.55 0)
+			(effects
+				(font
+					(size 1.27 1.27)
+				)
+				(hide yes)
+			)
+		)
+		(property "Description" "Power symbol creates a global label with name \"GND\" , ground"
+			(at 121.92 82.55 0)
+			(effects
+				(font
+					(size 1.27 1.27)
+				)
+				(hide yes)
+			)
+		)
+		(pin "1"
+		)
+		(instances
+			(project "OptiTrackMarker"
+				(path "/1ee121e3-f00f-41e9-9f71-839fc9072ed1/1c3e6d0c-0655-4cbd-ac01-be204861f2c1"
+					(reference "#PWR011")
+					(unit 1)
+				)
